Commit message: Tried to include ackermann

File: description/rover_core.xacro (robot description, xacro)
@@ -28,7 +28,10 @@
         </collisions>
         <xacro:inertial_box mass="0.5" x="0.6" y="0.4" z="0.2" >
-            <origin xyz="0 0 0.1" rpy="0 0 0" />
+            <origin xyz="0 0 0" rpy="0 0 0" />
         </xacro:inertial_box>
     </link>
+    <gazebo reference="chassis">
+        <material>Gazebo/White</material>
+    </gazebo>
     <!--    LIDAR   -->
     <link name="lidar_link">
@@ -50,4 +53,7 @@
         </xacro:inertial_cylinder>
     </link>
+    <gazebo reference="lidar_link">
+        <material>Gazebo/Blue</material>
+    </gazebo>
     <!--    RUEDAS   -->                        <!--     Definir dimensiones ruedas         -->
     <link name="front_right_wheel">
@@ -69,4 +75,7 @@
         </xacro:inertial_cylinder>
     </link>
+    <gazebo reference="front_right_wheel">
+        <material>Gazebo/Grey</material>
+    </gazebo>
     <link name="middle_right_wheel">
         <visual>
@@ -87,4 +96,7 @@
         </xacro:inertial_cylinder>
     </link>
+    <gazebo reference="middle_right_wheel">
+        <material>Gazebo/Grey</material>
+    </gazebo>
     <link name="rear_right_wheel">
         <visual>
@@ -105,4 +117,7 @@
         </xacro:inertial_cylinder>
     </link>
+    <gazebo reference="rear_right_wheel">
+        <material>Gazebo/Grey</material>
+    </gazebo>
     <link name="front_left_wheel">
         <visual>
@@ -123,4 +138,7 @@
         </xacro:inertial_cylinder>
     </link>
+    <gazebo reference="front_left_wheel">
+        <material>Gazebo/Grey</material>
+    </gazebo>
     <link name="middle_left_wheel">
         <visual>
@@ -141,4 +159,7 @@
         </xacro:inertial_cylinder>
     </link>
+    <gazebo reference="middle_left_wheel">
+        <material>Gazebo/Grey</material>
+    </gazebo>
     <link name="rear_left_wheel">
         <visual>
@@ -159,24 +180,82 @@
         </xacro:inertial_cylinder>
     </link>
+    <gazebo reference="rear_left_wheel">
+        <material>Gazebo/Grey</material>
+    </gazebo>
     <!--    STEERING    -->
     <link name="front_right_steering">
         <visual>
-            <origin xyz="0 0 0" rpy="0 0 0" />
-        </visual>
+            <geometry>
+                <cylinder radius="0.00001" length="0.00005"/>
+            </geometry>
+        </visual>
+        <collision>
+            <geometry>
+                <cylinder radius="0.00001" length="0.00005"/>
+            </geometry>
+        </collision>
+        <xacro:inertial_cylinder mass="0.00001" length="0.000005" radius="0.00001">
+            <origin xyz="0 0 0" rpy="0 0 0" />
+        </xacro:inertial_cylinder>
     </link>
     <link name="rear_right_steering">
         <visual>
-            <origin xyz="0 0 0" rpy="0 0 0" />
-        </visual>
+            <geometry>
+                <cylinder radius="0.00001" length="0.00005"/>
+            </geometry>
+        </visual>
+        <collision>
+            <geometry>
+                <cylinder radius="0.00001" length="0.00005"/>
+            </geometry>
+        </collision>
+        <xacro:inertial_cylinder mass="0.00001" length="0.000005" radius="0.00001">
+            <origin xyz="0 0 0" rpy="0 0 0" />
+        </xacro:inertial_cylinder>
     </link>
     <link name="front_left_steering">
         <visual>
-            <origin xyz="0 0 0" rpy="0 0 0" />
-        </visual>
+            <geometry>
+                <cylinder radius="0.00001" length="0.00005"/>
+            </geometry>
+        </visual>
+        <collision>
+            <geometry>
+                <cylinder radius="0.00001" length="0.00005"/>
+            </geometry>
+        </collision>
+        <xacro:inertial_cylinder mass="0.00001" length="0.000005" radius="0.00001">
+            <origin xyz="0 0 0" rpy="0 0 0" />
+        </xacro:inertial_cylinder>
     </link>
     <link name="rear_left_steering">
         <visual>
-            <origin xyz="0 0 0" rpy="0 0 0" />
-        </visual>
+            <geometry>
+                <cylinder radius="0.00001" length="0.00005"/>
+            </geometry>
+        </visual>
+        <collision>
+            <geometry>
+                <cylinder radius="0.00001" length="0.00005"/>
+            </geometry>
+        </collision>
+        <xacro:inertial_cylinder mass="0.00001" length="0.000005" radius="0.00001">
+            <origin xyz="0 0 0" rpy="0 0 0" />
+        </xacro:inertial_cylinder>
+    </link>
+    <link name="steering_wheel">
+        <visual>
+            <geometry>
+                <cylinder radius="0.00001" length="0.00005"/>
+            </geometry>
+        </visual>
+        <collision>
+            <geometry>
+                <cylinder radius="0.00001" length="0.00005"/>
+            </geometry>
+        </collision>
+        <xacro:inertial_cylinder mass="0.00001" length="0.000005" radius="0.00001">
+            <origin xyz="0 0 0" rpy="0 0 0" />
+        </xacro:inertial_cylinder>
     </link>
     <!--     JOINTS                   ### MEDIDAS A DEFINIR ###-->
@@ -191,4 +270,11 @@
         <origin xyz="0 0 0.125" rpy="0 0 0" />
     </joint>
+    <joint name="steering_wheel_joint" type="revolute">
+        <parent link="chassis" />
+        <child link="steering_wheel" />
+        <origin xyz="0 0 0.30" rpy="0 0 0" /> <!-- Cuanto sobresale sobre el eje z-->
+        <axis xyz="0 0 1" />
+        <limit lower="-1.57" upper="1.57" effort="10" velocity="1" />
+    </joint>
     <joint name="front_right_steering_joint" type="revolute">
         <parent link="chassis" />

File: description/rover_sener.urdf.xacro (robot description, xacro)
@@ -2,3 +2,4 @@
 <robot xmlns:xacro="http://www.ros.org/wiki/xacro"  name="rover_sener">
     <xacro:include filename="rover_core.xacro" />
+    <xacro:include filename="gazebo_control.xacro" />
 </robot>
